Commit message: Separete code between xacro and urdf file

File: urdf/vss_robot.xacro (robot description, xacro)
@@ -1,6 +1,3 @@
 <?xml version="1.0" encoding="utf-8"?>
-<!-- This URDF was automatically created by SolidWorks to URDF Exporter! Originally created by Stephen Brawner (brawner@gmail.com)
-     Commit Version: 1.5.1-0-g916b5db  Build Version: 1.5.7152.31018
-     For more information, please see http://wiki.ros.org/sw_urdf_exporter -->
 <robot name="vss_robot" xmlns:xacro="http://www.ros.org/wiki/xacro">
   <!-- Import all Gazebo-customization elements, including Gazebo colors -->
@@ -8,156 +5,10 @@
   <!-- Import Rviz colors -->
   <xacro:include filename="$(find vss_robot)/urdf/materials.xacro" />
-  <!-- <xacro:include filename="package://vss_robot/urdf/materials.xacro" /> -->
-  <link
-    name="Corpo">
-    <inertial>
-      <origin
-        xyz="0.00077374 1.5272E-09 -0.038284"
-        rpy="0 0 0" />
-      <mass
-        value="0.12206" />
-      <inertia
-        ixx="5.6918E-05"
-        ixy="-5.9966E-09"
-        ixz="-4.914E-06"
-        iyy="6.5745E-05"
-        iyz="4.347E-13"
-        izz="9.8955E-05" />
-    </inertial>
-    <visual>
-      <origin
-        xyz="0 0 0"
-        rpy="0 0 0" />
-      <geometry>
-        <mesh
-          filename="package://vss_robot/meshes/Corpo.STL" />
-      </geometry>
-      <material
-        name="abs">
-        <color
-          rgba="1 1 1 1" />
-      </material>
-    </visual>
-    <collision>
-      <origin
-        xyz="0 0 0"
-        rpy="0 0 0" />
-      <geometry>
-        <mesh
-          filename="package://vss_robot/meshes/Corpo.STL" />
-      </geometry>
-    </collision>
-  </link>
-  <link
-    name="RodaEsq">
-    <inertial>
-      <origin
-        xyz="2.9834E-06 -1.8789E-06 -0.0037178"
-        rpy="0 0 0" />
-      <mass
-        value="0.017155" />
-      <inertia
-        ixx="4.3502E-06"
-        ixy="-1.1633E-10"
-        ixz="1.2876E-17"
-        iyy="4.3501E-06"
-        iyz="-1.0322E-16"
-        izz="8.5226E-06" />
-    </inertial>
-    <visual>
-      <origin
-        xyz="0 0 0"
-        rpy="0 0 0" />
-      <geometry>
-        <mesh
-          filename="package://vss_robot/meshes/RodaEsq.STL" />
-      </geometry>
-      <material
-        name="plastic">
-        <color
-          rgba="0.69804 0.69804 0.69804 1" />
-      </material>
-    </visual>
-    <collision>
-      <origin
-        xyz="0 0 0"
-        rpy="0 0 0" />
-      <geometry>
-        <mesh
-          filename="package://vss_robot/meshes/RodaEsq.STL" />
-      </geometry>
-    </collision>
-  </link>
-  <joint
-    name="RodaEsq"
-    type="continuous">
-    <origin
-      xyz="-0.0052523 0.0362 -0.038501"
-      rpy="1.5708 1.0338 3.1416" />
-    <parent
-      link="Corpo" />
-    <child
-      link="RodaEsq" />
-    <axis
-      xyz="0 0 1" />
-    <limit
-      effort="0"
-      velocity="1000" />
-  </joint>
-  <link
-    name="RodaDir">
-    <inertial>
-      <origin
-        xyz="-4.51996190059534E-08 -3.52311700728414E-06 -0.00371783525923547"
-        rpy="0 0 0" />
-      <mass
-        value="0.0171546672764287" />
-      <inertia
-        ixx="4.35000652569962E-06"
-        ixy="1.60203597654766E-15"
-        ixz="-8.29550066436761E-17"
-        iyy="4.35027517811247E-06"
-        iyz="6.27650064229579E-17"
-        izz="8.52255775209774E-06" />
-    </inertial>
-    <visual>
-      <origin
-        xyz="0 0 0"
-        rpy="0 0 0" />
-      <geometry>
-        <mesh
-          filename="package://vss_robot/meshes/RodaDir.STL" />
-      </geometry>
-      <material
-        name="plastic">
-        <color
-          rgba="0.698039215686274 0.698039215686274 0.698039215686274 1" />
-      </material>
-    </visual>
-    <collision>
-      <origin
-        xyz="0 0 0"
-        rpy="0 0 0" />
-      <geometry>
-        <mesh
-          filename="package://vss_robot/meshes/RodaDir.STL" />
-      </geometry>
-    </collision>
-  </link>
-  <joint
-    name="RodaDir"
-    type="continuous">
-    <origin
-      xyz="-0.0052489 -0.0362 -0.038501"
-      rpy="1.5708 -0.2572 0" />
-    <parent
-      link="Corpo" />
-    <child
-      link="RodaDir" />
-    <axis
-      xyz="0 0 -1" />
-    <limit
-      effort="0"
-      velocity="1000" />
-  </joint>
+  <!-- Code exported from SolidWorks -->
+  <xacro:include filename="$(find vss_robot)/urdf/vss_robot.urdf" />
+  <gazebo>
+    <plugin name="gazebo_ros_control" filename="libgazebo_ros_control.so">
+      <robotNamespace>/</robotNamespace>
+    </plugin>
+  </gazebo>
 </robot>

Commit message: Fix SDL inertial warning

File: urdf/vss_robot.xacro (robot description, xacro)
@@ -1,4 +1,9 @@
 <?xml version="1.0" encoding="utf-8"?>
 <robot name="vss_robot" xmlns:xacro="http://www.ros.org/wiki/xacro">
+  <link name="base_link"/>
+  <joint name="base_joint" type="fixed">
+    <parent link="base_link"/>
+    <child link="Corpo"/>
+  </joint>
   <!-- Import all Gazebo-customization elements, including Gazebo colors -->
   <xacro:include filename="$(find vss_robot)/urdf/vss_robot.gazebo" />

Commit message: Fix link name change

File: urdf/vss_robot.xacro (robot description, xacro)
@@ -4,5 +4,5 @@
   <joint name="base_joint" type="fixed">
     <parent link="base_link"/>
-    <child link="Corpo"/>
+    <child link="corpo"/>
   </joint>
   <!-- Import all Gazebo-customization elements, including Gazebo colors -->

Commit message: :recycle: Refactor xacro files for team_number param

File: urdf/vss_robot.xacro (robot description, xacro)
@@ -2,4 +2,5 @@
 <robot name="vss_robot" xmlns:xacro="http://www.ros.org/wiki/xacro">
   <xacro:arg name="robot_number" default="0" />
+  <xacro:arg name="team_number" default="0" />
   <link name="base_link"/>
   <joint name="base_joint" type="fixed">

File: urdf/vss_team.xacro (robot description, xacro)
@@ -2,5 +2,7 @@
 <robot xmlns:xacro="http://www.ros.org/wiki/xacro">
     <xacro:arg name="robot_number" default="0" />
+    <xacro:arg name="team_number" default="0" />
     <xacro:property name="robot_number" value="$(arg robot_number)" />
+    <xacro:property name="team_number" value="$(arg team_number)" />
     <!-- Set common colors -->
     <gazebo reference="tile_sup_dir_link">
@@ -10,8 +12,34 @@
         <material>Gazebo/Black</material>
     </gazebo>
-    <gazebo reference="tile_inf_dir_link">
-        <material>Gazebo/Yellow</material>
-    </gazebo>
-    <!-- Set specific colors -->
+    <!-- Set teams configuration -->
+    <xacro:if value="${team_number == 0}">
+        <gazebo reference="tile_inf_dir_link">
+            <material>Gazebo/Yellow</material>
+        </gazebo>
+        <gazebo reference="corpo">
+            <material>Gazebo/White</material>
+        </gazebo>
+        <gazebo reference="roda_dir_link">
+            <material>Gazebo/Green</material>
+        </gazebo>
+        <gazebo reference="roda_esq_link">
+            <material>Gazebo/Green</material>
+        </gazebo>
+    </xacro:if>
+    <xacro:if value="${team_number == 1}">
+        <gazebo reference="tile_inf_dir_link">
+            <material>Gazebo/Blue</material>
+        </gazebo>
+        <gazebo reference="corpo">
+            <material>Gazebo/Grey</material>
+        </gazebo>
+        <gazebo reference="roda_dir_link">
+            <material>Gazebo/Red</material>
+        </gazebo>
+        <gazebo reference="roda_esq_link">
+            <material>Gazebo/Red</material>
+        </gazebo>
+    </xacro:if>
+    <!-- Set robots colors -->
     <xacro:if value="${robot_number == 0}">
         <gazebo reference="chapeu_link">
@@ -38,73 +66,3 @@
         </gazebo>
     </xacro:if>
-        <!-- <xacro:if value="${robot_number == 3}">
-            <material>Gazebo/Black</material>
-        </xacro:if>
-        <xacro:if value="${robot_number == 4}">
-            <material>Gazebo/Yellow</material>
-        </xacro:if>
-        <xacro:if value="${robot_number == 5}">
-            <material>Gazebo/Orange</material>
-        </xacro:if>
-    </gazebo> -->
-    <gazebo reference="corpo">
-        <xacro:if value="${robot_number == 0}">
-            <material>Gazebo/White</material>
-        </xacro:if>
-        <xacro:if value="${robot_number == 1}">
-            <material>Gazebo/White</material>
-        </xacro:if>
-        <xacro:if value="${robot_number == 2}">
-            <material>Gazebo/White</material>
-        </xacro:if>
-        <xacro:if value="${robot_number == 3}">
-            <material>Gazebo/Grey</material>
-        </xacro:if>
-        <xacro:if value="${robot_number == 4}">
-            <material>Gazebo/Grey</material>
-        </xacro:if>
-        <xacro:if value="${robot_number == 5}">
-            <material>Gazebo/Grey</material>
-        </xacro:if>
-    </gazebo>
-    <gazebo reference="roda_dir_link">
-        <xacro:if value="${robot_number == 0}">
-            <material>Gazebo/Green</material>
-        </xacro:if>
-        <xacro:if value="${robot_number == 1}">
-            <material>Gazebo/Green</material>
-        </xacro:if>
-        <xacro:if value="${robot_number == 2}">
-            <material>Gazebo/Green</material>
-        </xacro:if>
-        <xacro:if value="${robot_number == 3}">
-            <material>Gazebo/Red</material>
-        </xacro:if>
-        <xacro:if value="${robot_number == 4}">
-            <material>Gazebo/Red</material>
-        </xacro:if>
-        <xacro:if value="${robot_number == 5}">
-            <material>Gazebo/Red</material>
-        </xacro:if>
-    </gazebo>
-    <gazebo reference="roda_esq_link">
-        <xacro:if value="${robot_number == 0}">
-            <material>Gazebo/Green</material>
-        </xacro:if>
-        <xacro:if value="${robot_number == 1}">
-            <material>Gazebo/Green</material>
-        </xacro:if>
-        <xacro:if value="${robot_number == 2}">
-            <material>Gazebo/Green</material>
-        </xacro:if>
-        <xacro:if value="${robot_number == 3}">
-            <material>Gazebo/Red</material>
-        </xacro:if>
-        <xacro:if value="${robot_number == 4}">
-            <material>Gazebo/Red</material>
-        </xacro:if>
-        <xacro:if value="${robot_number == 5}">
-            <material>Gazebo/Red</material>
-        </xacro:if>
-    </gazebo>
 </robot>
