Commit message: Change var names to follow convention

File: urdf/vss_robot.urdf (robot description, URDF)
Before this commit: robot vss_robot, 3 links, 2 joints
Links:
- removed link RodaDir
- removed link RodaEsq
- added link roda_dir_link, mass 0.0171546672764287; collision mesh filename=package://vss_robot/meshes/RodaDir.STL; visual mesh filename=package://vss_robot/meshes/RodaDir.STL
- added link roda_esq_link, mass 0.017155; collision mesh filename=package://vss_robot/meshes/RodaEsq.STL; visual mesh filename=package://vss_robot/meshes/RodaEsq.STL
Joints:
- removed joint RodaDir
- removed joint RodaEsq
- added joint roda_dir_joint: type continuous, parent Corpo, child roda_dir_link, origin xyz=-0.0052489 -0.0362 -0.038501 rpy=1.5708 -0.2572 0, axis 0 0 -1, limit effort=0 velocity=1000
- added joint roda_esq_joint: type continuous, parent Corpo, child roda_esq_link, origin xyz=-0.0052523 0.0362 -0.038501 rpy=1.5708 1.0338 3.1416, axis 0 0 1, limit effort=0 velocity=1000

Commit message: Update robot model
Add functional motors to the robot model

File: urdf/vss_robot.urdf (robot description, URDF)
Before this commit: robot vss_robot, 3 links, 2 joints
Joints:
- joint roda_dir_joint: limit effort=0 velocity=1000 -> (none)
- joint roda_esq_joint: limit effort=0 velocity=1000 -> (none)

File: urdf/vss_robot.xacro (robot description, xacro)
@@ -7,4 +7,9 @@
   <!-- Code exported from SolidWorks -->
   <xacro:include filename="$(find vss_robot)/urdf/vss_robot.urdf" />
+  <!-- Definition of motor -->
+  <xacro:include filename="$(find vss_robot)/urdf/motor.xacro"/>
+  <xacro:motor side="esq" gear_rate="1"/>
+  <xacro:motor side="dir" gear_rate="1"/>
+  <!-- Load gazebo plugin to control the robot -->
   <gazebo>
     <plugin name="gazebo_ros_control" filename="libgazebo_ros_control.so">

Commit message: Update model from SolidWorks

File: urdf/vss_robot.urdf (robot description, URDF)
Before this commit: robot vss_robot, 3 links, 2 joints
Links:
- removed link Corpo
- added link chapeu_link, mass 0.022727; collision mesh filename=package://vss_simulation/meshes/chapeu_link.STL; visual mesh filename=package://vss_simulation/meshes/chapeu_link.STL
- added link corpo, mass 0.11426; collision mesh filename=package://vss_simulation/meshes/corpo.STL; visual mesh filename=package://vss_simulation/meshes/corpo.STL
- link roda_dir_link: mass 0.0171546672764287 -> 0.017155; geometry collision mesh filename=package://vss_simulation/meshes/roda_dir_link.STL; visual mesh filename=package://vss_simulation/meshes/roda_dir_link.STL
- link roda_esq_link: geometry collision mesh filename=package://vss_simulation/meshes/roda_esq_link.STL; visual mesh filename=package://vss_simulation/meshes/roda_esq_link.STL
Joints:
- added joint chapeu_joint: type fixed, parent corpo, child chapeu_link, origin xyz=0 -0.0105 0.0653 rpy=0 0 0, axis 0 0 0
- joint roda_dir_joint: origin xyz=-0.0052489 -0.0362 -0.038501 rpy=1.5708 -0.2572 0 -> xyz=0.032251 -0.0092 0.026799 rpy=1.5708 -0.2572 0; parent Corpo -> corpo
- joint roda_esq_joint: origin xyz=-0.0052523 0.0362 -0.038501 rpy=1.5708 1.0338 3.1416 -> xyz=0.032248 0.0632 0.026799 rpy=1.5708 -0.013398 3.1416; parent Corpo -> corpo

Commit message: :bento: Update URDF model from SolidWorks

File: urdf/vss_robot.urdf (robot description, URDF)
Before this commit: robot vss_robot, 4 links, 3 joints
Links:
- added link tile_inf_dir_link, mass 0.002109375; collision mesh filename=package://vss_simulation/meshes/tile_inf_dir_link.STL; visual mesh filename=package://vss_simulation/meshes/tile_inf_dir_link.STL
- added link tile_inf_esq_link, mass 0.002109375; collision mesh filename=package://vss_simulation/meshes/tile_inf_esq_link.STL; visual mesh filename=package://vss_simulation/meshes/tile_inf_esq_link.STL
- added link tile_sup_dir_link, mass 0.002109375; collision mesh filename=package://vss_simulation/meshes/tile_sup_dir_link.STL; visual mesh filename=package://vss_simulation/meshes/tile_sup_dir_link.STL
- added link tile_sup_esq_link, mass 0.002109375; collision mesh filename=package://vss_simulation/meshes/tile_sup_esq_link.STL; visual mesh filename=package://vss_simulation/meshes/tile_sup_esq_link.STL
- link chapeu_link: mass 0.022727 -> 0.0141218190526683
- link corpo: mass 0.11426 -> 0.114255136924402
- link roda_esq_link: mass 0.017155 -> 0.0171546672764287
Joints:
- added joint tile_inf_dir_joint: type fixed, parent chapeu_link, child tile_inf_dir_link, origin xyz=0 0 0 rpy=0 0 0, axis 0 0 0
- added joint tile_inf_esq_joint: type fixed, parent chapeu_link, child tile_inf_esq_link, origin xyz=0 0 0 rpy=0 0 0, axis 0 0 0
- added joint tile_sup_dir_joint: type fixed, parent chapeu_link, child tile_sup_dir_link, origin xyz=0 0 0 rpy=0 0 0, axis 0 0 0
- added joint tile_sup_esq_joint: type fixed, parent chapeu_link, child tile_sup_esq_link, origin xyz=0 0 0 rpy=0 0 0, axis 0 0 0
- joint chapeu_joint: origin xyz=0 -0.0105 0.0653 rpy=0 0 0 -> xyz=0.00525000000000002 0 0.0653 rpy=0 0 0
- joint roda_dir_joint: origin xyz=0.032251 -0.0092 0.026799 rpy=1.5708 -0.2572 0 -> xyz=0 -0.0362 0.0267989207102477 rpy=1.5707963267949 -0.257204591428631 0
- joint roda_esq_joint: origin xyz=0.032248 0.0632 0.026799 rpy=1.5708 -0.013398 3.1416 -> xyz=0 0.0362 0.02679871482879 rpy=1.5707963267949 -0.0133976378081295 3.14159265358979

File: urdf/vss_team.xacro (robot description, xacro)
@@ -3,14 +3,38 @@
     <xacro:arg name="robot_number" default="0" />
     <xacro:property name="robot_number" value="$(arg robot_number)" />
-    <gazebo reference="chapeu_link">
-        <xacro:if value="${robot_number == 0}">
+    <!-- Set common colors -->
+    <gazebo reference="tile_sup_dir_link">
+        <material>Gazebo/Black</material>
+    </gazebo>
+    <gazebo reference="tile_inf_esq_link">
+        <material>Gazebo/Black</material>
+    </gazebo>
+    <gazebo reference="tile_inf_dir_link">
+        <material>Gazebo/Yellow</material>
+    </gazebo>
+    <!-- Set specific colors -->
+    <xacro:if value="${robot_number == 0}">
+        <gazebo reference="chapeu_link">
             <material>Gazebo/Black</material>
-        </xacro:if>
-        <xacro:if value="${robot_number == 1}">
-            <material>Gazebo/Yellow</material>
-        </xacro:if>
-        <xacro:if value="${robot_number == 2}">
+        </gazebo>
+        <gazebo reference="tile_sup_esq_link">
+            <material>Gazebo/Purple</material>
+        </gazebo>
+    </xacro:if>
+    <xacro:if value="${robot_number == 1}">
+        <gazebo reference="chapeu_link">
+            <material>Gazebo/Black</material>
+        </gazebo>
+        <gazebo reference="tile_sup_esq_link">
             <material>Gazebo/Orange</material>
-        </xacro:if>
-    </gazebo>
+        </gazebo>
+    </xacro:if>
+    <xacro:if value="${robot_number == 2}">
+        <gazebo reference="chapeu_link">
+            <material>Gazebo/Black</material>
+        </gazebo>
+        <gazebo reference="tile_sup_esq_link">
+            <material>Gazebo/Green</material>
+        </gazebo>
+    </xacro:if>
 </robot>

Commit message: :alembic: Set dynamics parameters for wheels joints

File: urdf/vss_robot.urdf (robot description, URDF)
Before this commit: robot vss_simulation, 8 links, 7 joints
Joints:
- joint roda_dir_joint: limit (none) -> effort=108e-3 velocity=100
- joint roda_esq_joint: limit (none) -> effort=108e-3 velocity=100
