Commit message: Add new launch file: simulation_match.launch

File: urdf/vss_team.xacro (robot description, xacro)
@@ -13,4 +13,73 @@
             <material>Gazebo/Orange</material>
         </xacro:if>
+        <xacro:if value="${robot_number == 3}">
+            <material>Gazebo/Black</material>
+        </xacro:if>
+        <xacro:if value="${robot_number == 4}">
+            <material>Gazebo/Yellow</material>
+        </xacro:if>
+        <xacro:if value="${robot_number == 5}">
+            <material>Gazebo/Orange</material>
+        </xacro:if>
+    </gazebo>
+    <gazebo reference="corpo">
+        <xacro:if value="${robot_number == 0}">
+            <material>Gazebo/White</material>
+        </xacro:if>
+        <xacro:if value="${robot_number == 1}">
+            <material>Gazebo/White</material>
+        </xacro:if>
+        <xacro:if value="${robot_number == 2}">
+            <material>Gazebo/White</material>
+        </xacro:if>
+        <xacro:if value="${robot_number == 3}">
+            <material>Gazebo/Grey</material>
+        </xacro:if>
+        <xacro:if value="${robot_number == 4}">
+            <material>Gazebo/Grey</material>
+        </xacro:if>
+        <xacro:if value="${robot_number == 5}">
+            <material>Gazebo/Grey</material>
+        </xacro:if>
+    </gazebo>
+    <gazebo reference="roda_dir_link">
+        <xacro:if value="${robot_number == 0}">
+            <material>Gazebo/Green</material>
+        </xacro:if>
+        <xacro:if value="${robot_number == 1}">
+            <material>Gazebo/Green</material>
+        </xacro:if>
+        <xacro:if value="${robot_number == 2}">
+            <material>Gazebo/Green</material>
+        </xacro:if>
+        <xacro:if value="${robot_number == 3}">
+            <material>Gazebo/Red</material>
+        </xacro:if>
+        <xacro:if value="${robot_number == 4}">
+            <material>Gazebo/Red</material>
+        </xacro:if>
+        <xacro:if value="${robot_number == 5}">
+            <material>Gazebo/Red</material>
+        </xacro:if>
+    </gazebo>
+    <gazebo reference="roda_esq_link">
+        <xacro:if value="${robot_number == 0}">
+            <material>Gazebo/Green</material>
+        </xacro:if>
+        <xacro:if value="${robot_number == 1}">
+            <material>Gazebo/Green</material>
+        </xacro:if>
+        <xacro:if value="${robot_number == 2}">
+            <material>Gazebo/Green</material>
+        </xacro:if>
+        <xacro:if value="${robot_number == 3}">
+            <material>Gazebo/Red</material>
+        </xacro:if>
+        <xacro:if value="${robot_number == 4}">
+            <material>Gazebo/Red</material>
+        </xacro:if>
+        <xacro:if value="${robot_number == 5}">
+            <material>Gazebo/Red</material>
+        </xacro:if>
     </gazebo>
 </robot>

Commit message: :bento: Configure color of robots hats

File: urdf/vss_team.xacro (robot description, xacro)
@@ -26,4 +26,29 @@
             <material>Gazebo/Green</material>
         </gazebo>
+        <!-- Set robots colors -->
+        <xacro:if value="${robot_number == 0}">
+            <gazebo reference="chapeu_link">
+                <material>Gazebo/Black</material>
+            </gazebo>
+            <gazebo reference="tile_sup_esq_link">
+                <material>Gazebo/Purple</material>
+            </gazebo>
+        </xacro:if>
+        <xacro:if value="${robot_number == 1}">
+            <gazebo reference="chapeu_link">
+                <material>Gazebo/Black</material>
+            </gazebo>
+            <gazebo reference="tile_sup_esq_link">
+                <material>Gazebo/Red</material>
+            </gazebo>
+        </xacro:if>
+        <xacro:if value="${robot_number == 2}">
+            <gazebo reference="chapeu_link">
+                <material>Gazebo/Black</material>
+            </gazebo>
+            <gazebo reference="tile_sup_esq_link">
+                <material>Gazebo/Green</material>
+            </gazebo>
+        </xacro:if>  <!-- /Set robots colors -->
     </xacro:if>
     <xacro:if value="${team_number == 1}">
@@ -40,29 +65,29 @@
             <material>Gazebo/Red</material>
         </gazebo>
-    </xacro:if>
-    <!-- Set robots colors -->
-    <xacro:if value="${robot_number == 0}">
-        <gazebo reference="chapeu_link">
-            <material>Gazebo/Black</material>
-        </gazebo>
-        <gazebo reference="tile_sup_esq_link">
-            <material>Gazebo/Purple</material>
-        </gazebo>
-    </xacro:if>
-    <xacro:if value="${robot_number == 1}">
-        <gazebo reference="chapeu_link">
-            <material>Gazebo/Black</material>
-        </gazebo>
-        <gazebo reference="tile_sup_esq_link">
-            <material>Gazebo/Orange</material>
-        </gazebo>
-    </xacro:if>
-    <xacro:if value="${robot_number == 2}">
-        <gazebo reference="chapeu_link">
-            <material>Gazebo/Black</material>
-        </gazebo>
-        <gazebo reference="tile_sup_esq_link">
-            <material>Gazebo/Green</material>
-        </gazebo>
+        <!-- Set robots colors -->
+        <xacro:if value="${robot_number == 0}">
+            <gazebo reference="chapeu_link">
+                <material>Gazebo/Black</material>
+            </gazebo>
+            <gazebo reference="tile_sup_esq_link">
+                <material>Gazebo/SkyBlue</material>
+            </gazebo>
+        </xacro:if>
+        <xacro:if value="${robot_number == 1}">
+            <gazebo reference="chapeu_link">
+                <material>Gazebo/Black</material>
+            </gazebo>
+            <gazebo reference="tile_sup_esq_link">
+                <material>Gazebo/Turquoise</material>
+            </gazebo>
+        </xacro:if>
+        <xacro:if value="${robot_number == 2}">
+            <gazebo reference="chapeu_link">
+                <material>Gazebo/Black</material>
+            </gazebo>
+            <gazebo reference="tile_sup_esq_link">
+                <material>Gazebo/Indigo</material>
+            </gazebo>
+        </xacro:if>  <!-- /Set robots colors -->
     </xacro:if>
 </robot>

Commit message: Change hat color pattern

File: urdf/vss_team.xacro (robot description, xacro)
@@ -5,16 +5,7 @@
     <xacro:property name="robot_number" value="$(arg robot_number)" />
     <xacro:property name="team_number" value="$(arg team_number)" />
-    <!-- Set common colors -->
-    <gazebo reference="tile_sup_dir_link">
-        <material>Gazebo/Black</material>
-    </gazebo>
-    <gazebo reference="tile_inf_esq_link">
-        <material>Gazebo/Black</material>
-    </gazebo>
-    <!-- Set teams configuration -->
+    <xacro:include filename="$(find vss_simulation)/urdf/hat_colors.xacro"/>
+    <!-- Set team configuration -->
     <xacro:if value="${team_number == 0}">
-        <gazebo reference="tile_inf_dir_link">
-            <material>Gazebo/Yellow</material>
-        </gazebo>
         <gazebo reference="corpo">
             <material>Gazebo/White</material>
@@ -27,33 +18,16 @@
         </gazebo>
         <!-- Set robots colors -->
-        <xacro:if value="${robot_number == 0}">
-            <gazebo reference="chapeu_link">
-                <material>Gazebo/Black</material>
-            </gazebo>
-            <gazebo reference="tile_sup_esq_link">
-                <material>Gazebo/Purple</material>
-            </gazebo>
-        </xacro:if>
         <xacro:if value="${robot_number == 1}">
-            <gazebo reference="chapeu_link">
-                <material>Gazebo/Black</material>
-            </gazebo>
-            <gazebo reference="tile_sup_esq_link">
-                <material>Gazebo/Red</material>
-            </gazebo>
+            <xacro:hat_colors team_color="Gazebo/Yellow" robot_color="Gazebo/Purple" />
         </xacro:if>
         <xacro:if value="${robot_number == 2}">
-            <gazebo reference="chapeu_link">
-                <material>Gazebo/Black</material>
-            </gazebo>
-            <gazebo reference="tile_sup_esq_link">
-                <material>Gazebo/Green</material>
-            </gazebo>
+            <xacro:hat_colors team_color="Gazebo/Yellow" robot_color="Gazebo/Red" />
+        </xacro:if>
+        <xacro:if value="${robot_number == 3}">
+            <xacro:hat_colors team_color="Gazebo/Yellow" robot_color="Gazebo/Green" />
         </xacro:if>  <!-- /Set robots colors -->
-    </xacro:if>
+    </xacro:if> <!-- /Set team configuration -->
+    <!-- Set team configuration -->
     <xacro:if value="${team_number == 1}">
-        <gazebo reference="tile_inf_dir_link">
-            <material>Gazebo/Blue</material>
-        </gazebo>
         <gazebo reference="corpo">
             <material>Gazebo/Grey</material>
@@ -66,28 +40,13 @@
         </gazebo>
         <!-- Set robots colors -->
-        <xacro:if value="${robot_number == 0}">
-            <gazebo reference="chapeu_link">
-                <material>Gazebo/Black</material>
-            </gazebo>
-            <gazebo reference="tile_sup_esq_link">
-                <material>Gazebo/SkyBlue</material>
-            </gazebo>
-        </xacro:if>
         <xacro:if value="${robot_number == 1}">
-            <gazebo reference="chapeu_link">
-                <material>Gazebo/Black</material>
-            </gazebo>
-            <gazebo reference="tile_sup_esq_link">
-                <material>Gazebo/Turquoise</material>
-            </gazebo>
+            <xacro:hat_colors team_color="Gazebo/Blue" robot_color="Gazebo/SkyBlue" />
         </xacro:if>
         <xacro:if value="${robot_number == 2}">
-            <gazebo reference="chapeu_link">
-                <material>Gazebo/Black</material>
-            </gazebo>
-            <gazebo reference="tile_sup_esq_link">
-                <material>Gazebo/Indigo</material>
-            </gazebo>
+            <xacro:hat_colors team_color="Gazebo/Blue" robot_color="Gazebo/Turquoise" />
+        </xacro:if>
+        <xacro:if value="${robot_number == 3}">
+            <xacro:hat_colors team_color="Gazebo/Blue" robot_color="Gazebo/Indigo" />
         </xacro:if>  <!-- /Set robots colors -->
-    </xacro:if>
+    </xacro:if> <!-- /Set team configuration -->
 </robot>
