Commit message: :recycle: Remove redundant tags

File: urdf/generic_vss_robot.xacro (robot description, xacro)
@@ -4,4 +4,6 @@
   <xacro:arg name="robot_number" default="0" />
   <xacro:arg name="team_number" default="0" />
+  <xacro:property name="robot_number" value="$(arg robot_number)" />
+  <xacro:property name="team_number" value="$(arg team_number)" />
   <!-- Import all Gazebo-customization elements, except colors -->
   <xacro:include filename="$(find vss_simulation)/urdf/generic_vss_robot.gazebo" />

Commit message: 🔧  Change team_number param  to is_yellow

File: urdf/generic_vss_robot.xacro (robot description, xacro)
@@ -3,7 +3,7 @@
   xmlns:xacro="http://www.ros.org/wiki/xacro">
   <xacro:arg name="robot_number" default="0" />
-  <xacro:arg name="team_number" default="0" />
+  <xacro:arg name="is_yellow" default="0" />
   <xacro:property name="robot_number" value="$(arg robot_number)" />
-  <xacro:property name="team_number" value="$(arg team_number)" />
+  <xacro:property name="is_yellow" value="$(arg is_yellow)" />
   <!-- Import all Gazebo-customization elements, except colors -->
   <xacro:include filename="$(find vss_simulation)/urdf/generic_vss_robot.gazebo" />
