Commit message: :bento: Update textures for hat and sides

File: urdf/generic_vss_robot.urdf (robot description, URDF)
Before this commit: robot generic_vss_robot, 5 links, 4 joints
Links:
- added link parede_esq_link, mass 0.00918; collision mesh filename=package://generic_vss_robot/meshes/parede_esq_link.STL; visual box size=75e-3 2e-3 60e-3
- link chapeu_link: geometry collision box size=80e-3 80e-3 2e-3; visual box size=80e-3 80e-3 2e-3
- link parede_dir_link: geometry collision box size=75e-3 2e-3 60e-3; visual box size=75e-3 2e-3 60e-3
Joints:
- added joint parede_esq_joint: type fixed, parent base_link, child parede_esq_link, origin xyz=0 0 0 rpy=0 0 0, axis 0 0 0

Commit message: :ambulance: Fix launchfiles.
Co-authored-by: lucastrschneider <lucastrschneider@gmail.com>
Co-authored-by: Berbardo <bernardo.rcoutinho@gmail.com>

File: urdf/generic_vss_robot.urdf (robot description, URDF)
Before this commit: robot generic_vss_robot, 6 links, 5 joints
Links:
- link base_link: geometry collision mesh filename=package://vss_simulation/meshes/base_link.STL; visual mesh filename=package://vss_simulation/meshes/base_link.STL
- link parede_esq_link: geometry collision mesh filename=package://vss_simulation/meshes/parede_esq_link.STL; visual box size=75e-3 2e-3 60e-3
- link roda_dir_link: geometry collision mesh filename=package://vss_simulation/meshes/roda_dir_link.STL; visual mesh filename=package://vss_simulation/meshes/roda_dir_link.STL
- link roda_esq_link: geometry collision mesh filename=package://vss_simulation/meshes/roda_esq_link.STL; visual mesh filename=package://vss_simulation/meshes/roda_esq_link.STL

Commit message: :bento: Edit model joint according to ROS convention
See https://www.ros.org/reps/rep-0103.html for more details

File: urdf/generic_vss_robot.urdf (robot description, URDF)
Before this commit: robot generic_vss_robot, 6 links, 5 joints
Joints:
- joint roda_dir_joint: axis 0 -1 0 -> 0 1 0
- joint roda_esq_joint: axis 0 -1 0 -> 0 1 0

Commit message: Update motor parameters

File: urdf/generic_vss_robot.urdf (robot description, URDF)
Before this commit: robot generic_vss_robot, 6 links, 5 joints
Joints:
- joint roda_dir_joint: limit effort=0.108 velocity=100 -> effort=73e-3 velocity=68
- joint roda_esq_joint: limit effort=0.108 velocity=100 -> effort=73e-3 velocity=68

Commit message: ♻️ Update urdf model - Remove mesh from parede esq collision - Fix chapeu box size to match stl mesh

File: urdf/generic_vss_robot.urdf (robot description, URDF)
Before this commit: robot generic_vss_robot, 6 links, 5 joints
Links:
- link chapeu_link: geometry collision box size=75e-3 79e-3 2e-3; visual box size=75e-3 79e-3 2e-3
- link parede_esq_link: geometry collision box size=75e-3 2e-3 60e-3; visual box size=75e-3 2e-3 60e-3

Commit message: ⚡️ Replace wheels with primitives

File: urdf/generic_vss_robot.urdf (robot description, URDF)
Before this commit: robot generic_vss_robot, 6 links, 5 joints
Links:
- link roda_dir_link: geometry collision cylinder length=8e-3 radius=25e-3; visual cylinder length=8e-3 radius=25e-3
- link roda_esq_link: geometry collision cylinder length=8e-3 radius=25e-3; visual cylinder length=8e-3 radius=25e-3

Commit message: ⚡️ Improve model meshes - Remove unecessary collision links

File: urdf/generic_vss_robot.urdf (robot description, URDF)
Before this commit: robot generic_vss_robot, 6 links, 5 joints
Links:
- link base_link: geometry collision mesh filename=package://travesim/meshes/base_link_col.stl; visual mesh filename=package://travesim/meshes/base_link.stl
- link chapeu_link: geometry visual box size=75e-3 79e-3 2e-3
- link parede_dir_link: geometry visual box size=75e-3 2e-3 60e-3
- link parede_esq_link: geometry visual box size=75e-3 2e-3 60e-3
